Commit message: reorganize the xacro structure

File: ur5_arm_zell_description/urdf/ur5_structure.urdf.xacro (robot description, xacro)
@@ -1,59 +1,4 @@
 <?xml version="1.0"?>
-<robot xmlns:xacro="http://www.ros.org/wiki/xacro" name="ur5_base_zell">
-    <!-- Inertia parameters -->
-    <xacro:property name="base_mass" value="4.0" />  <!-- This mass might be incorrect -->
-    <xacro:property name="shoulder_mass" value="3.7000" />
-    <xacro:property name="upper_arm_mass" value="8.3930" />
-    <xacro:property name="forearm_mass" value="2.2750" />
-    <xacro:property name="wrist_1_mass" value="1.2190" />
-    <xacro:property name="wrist_2_mass" value="1.2190" />
-    <xacro:property name="wrist_3_mass" value="0.1879" />
-    <xacro:property name="shoulder_cog" value="0.0 0.00193 -0.02561" />
-    <xacro:property name="upper_arm_cog" value="0.0 -0.024201 0.2125" />
-    <xacro:property name="forearm_cog" value="0.0 0.0265 0.11993" />
-    <xacro:property name="wrist_1_cog" value="0.0 0.110949 0.01634" />
-    <xacro:property name="wrist_2_cog" value="0.0 0.0018 0.11099" />
-    <xacro:property name="wrist_3_cog" value="0.0 0.001159 0.0" />
-    <!-- Kinematic model -->
-    <!-- Properties from urcontrol.conf -->
-    <!--
-    DH for UR5
-    a = [0.00000, -0.42500, -0.39225,  0.00000,  0.00000,  0.0000]
-    d = [0.089159,  0.00000,  0.00000,  0.10915,  0.09465,  0.0823]
-    alpha = [ 1.570796327, 0, 0, 1.570796327, -1.570796327, 0 ]
-    q_home_offset = [0, -1.570796327, 0, -1.570796327, 0, 0]
-    joint_direction = [-1, -1, 1, 1, 1, 1]
-    mass = [3.7000, 8.3930, 2.2750, 1.2190, 1.2190, 0.1879]
-    center_of_mass = [ [0, -0.02561, 0.00193], [0.2125, 0, 0.11336], [0.11993, 0.0, 0.0265], [0, -0.0018, 0.01634], [0, 0.0018,0.01634], [0, 0, -0.001159] ]
-    -->
-    <xacro:property name="ur5_d1" value="0.089159" />
-    <xacro:property name="ur5_a2" value="-0.42500" />
-    <xacro:property name="ur5_a3" value="-0.39225" />
-    <xacro:property name="ur5_d4" value="0.10915" />
-    <xacro:property name="ur5_d5" value="0.09465" />
-    <xacro:property name="ur5_d6" value="0.0823" />
-    <!-- Arbitrary offsets for shoulder/elbow joints -->
-    <xacro:property name="shoulder_offset" value="0.13585" />  <!-- measured from model -->
-    <xacro:property name="elbow_offset" value="-0.1197" /> <!-- measured from model -->
-    <!-- link lengths used in model -->
-    <xacro:property name="shoulder_height" value="${ur5_d1}" />
-    <xacro:property name="upper_arm_length" value="${-ur5_a2}" />
-    <xacro:property name="forearm_length" value="${-ur5_a3}" />
-    <xacro:property name="wrist_1_length" value="${ur5_d4 - elbow_offset - shoulder_offset}" />
-    <xacro:property name="wrist_2_length" value="${ur5_d5}" />
-    <xacro:property name="wrist_3_length" value="${ur5_d6}" />
-    <!--property name="shoulder_height" value="0.089159" /-->
-    <!--property name="shoulder_offset" value="0.13585" /-->  <!-- shoulder_offset - elbow_offset + wrist_1_length = 0.10915 -->
-    <!--property name="upper_arm_length" value="0.42500" /-->
-    <!--property name="elbow_offset" value="0.1197" /-->       <!-- CAD measured -->
-    <!--property name="forearm_length" value="0.39225" /-->
-    <!--property name="wrist_1_length" value="0.093" /-->     <!-- CAD measured -->
-    <!--property name="wrist_2_length" value="0.09465" /-->   <!-- In CAD this distance is 0.930, but in the spec it is 0.09465 -->
-    <!--property name="wrist_3_length" value="0.0823" /-->
-    <xacro:property name="shoulder_radius" value="0.060" />   <!-- manually measured -->
-    <xacro:property name="upper_arm_radius" value="0.054" />  <!-- manually measured -->
-    <xacro:property name="elbow_radius" value="0.060" />      <!-- manually measured -->
-    <xacro:property name="forearm_radius" value="0.040" />    <!-- manually measured -->
-    <xacro:property name="wrist_radius" value="0.045" />      <!-- manually measured -->
+<robot xmlns:xacro="http://www.ros.org/wiki/xacro" name="ur5_structure">
     <xacro:macro name="cylinder_inertial" params="radius length mass *origin">
         <inertial>
@@ -65,6 +10,15 @@
         </inertial>
     </xacro:macro>
-    <!-- **************************************************** Define Links ******************************************************** -->
-    <xacro:macro name="ur5_robot" params="prefix joint_limited">
+    <xacro:macro name="force_torque_sensor" params="force_torque_sensor_link_name">
+        <sensor name="${force_torque_sensor_link_name}" type="force_torque">
+            <force_torque>
+                <frame>child</frame>
+                <measure_direction>child_to_parent</measure_direction>
+            </force_torque>
+            <update_rate>30.0</update_rate>
+		</sensor>
+    </xacro:macro>
+    <!-- Structure define -->
+    <xacro:macro name="ur5_robot" params="prefix joint_limited using_camera using_IMU using_laser using_force_torque">
         <link name="${prefix}base_link" >
             <visual>
@@ -96,4 +50,7 @@
                 <limit lower="${-pi}" upper="${pi}" effort="150.0" velocity="3.15"/>
             </xacro:if>
+            <xacro:if value="${using_force_torque}">
+                <xacro:force_torque_sensor force_torque_sensor_link_name="${prefix}shoulder_pan_sensor"/>
+            </xacro:if>
             <dynamics damping="0.5" friction="5.0"/>
         </joint>
@@ -127,4 +84,7 @@
 				<limit lower="${-pi}" upper="${pi}" effort="150.0" velocity="3.15"/>
 			</xacro:if>
+            <xacro:if value="${using_force_torque}">
+                <xacro:force_torque_sensor force_torque_sensor_link_name="${prefix}shoulder_lift_sensor"/>
+            </xacro:if>
 			<dynamics damping="0.5" friction="5.0"/>
 		</joint>
@@ -158,4 +118,7 @@
 				<limit lower="${-pi}" upper="${pi}" effort="150.0" velocity="3.15"/>
 			</xacro:if>
+            <xacro:if value="${using_force_torque}">
+                <xacro:force_torque_sensor force_torque_sensor_link_name="${prefix}elbow_sensor"/>
+            </xacro:if>
 			<dynamics damping="0.5" friction="5.0"/>
 		</joint>
@@ -189,4 +152,7 @@
 				<limit lower="${-pi}" upper="${pi}" effort="28.0" velocity="3.2"/>
 			</xacro:if>
+            <xacro:if value="${using_force_torque}">
+                <xacro:force_torque_sensor force_torque_sensor_link_name="${prefix}wrist_1_sensor"/>
+            </xacro:if>
 			<dynamics damping="0.5" friction="5.0"/>
 		</joint>
@@ -220,4 +186,7 @@
 				<limit lower="${-pi}" upper="${pi}" effort="28.0" velocity="3.2"/>
 			</xacro:if>
+            <xacro:if value="${using_force_torque}">
+                <xacro:force_torque_sensor force_torque_sensor_link_name="${prefix}wrist_2_sensor"/>
+            </xacro:if>
 			<dynamics damping="0.5" friction="5.0"/>
 		</joint>
@@ -251,4 +220,7 @@
 				<limit lower="${-pi}" upper="${pi}" effort="28.0" velocity="3.2"/>
 			</xacro:if>
+            <xacro:if value="${using_force_torque}">
+                <xacro:force_torque_sensor force_torque_sensor_link_name="${prefix}wrist_3_sensor"/>
+            </xacro:if>
 			<dynamics damping="0.5" friction="5.0"/>
 		</joint>
